File: BQ24650_1U_SolarChargerBoard.kicad_sch (KiCad schematic)
At the start: 36 parts, among them J1 Solar IO, J2 Battery IO, J3 CE_MPPSET, Q1 Q_NMOS_GDS, Q2 Q_NMOS_GDS, Q3 Q_NMOS_GDS, U1 BQ24650

Commit message: small changes
Parts:
- removed Rsr: R, symbol Device:R_Small
- added R12: RShunt, symbol Device:R_Small
- added R13: 0ohm, symbol Device:R_Small
- added TP1, TP10, TP11, TP12, TP2, TP3, TP4, TP5, TP6, TP7, TP8, TP9: TestPoint, symbol Connector:TestPoint
Connections:
- net -BATT is gone; now on net GND: C1.2, C2.2, C4.2, C6.2, C8.2, C9.2, J1.2 (Pin_2), J2.2 (Pin_2), Q2.3 (S), Q3.3 (S), R1.2, R10.1, R11.1, R4.1, U1.11 (GND), U1.17 (GND)
- net +BATT: now also R12.1, R13.1; no longer C7.2, U1.9 (SRN)
- net BTST: no longer Q1.1 (G), U1.15 (HIDRV)
- net CE: now also TP3.1
- net MPPSET: now also TP8.1
- net REGN: now also TP6.1
- net SRP: now also R12.2
- net STAT1: now also TP4.1
- net STAT2: now also TP5.1
- net VCC: now also TP1.1
- net VFB: now also TP10.1
- net VREF: now also TP7.1
- net at R4.2, RV2.1: now also TP12.1
- net at R1.1, RV1.1: now also TP11.1
- net TERM_EN: now reaches R11.2, U1.7 (TERM_EN)
- net TERM_EN: now also TP9.1
- net GND: now reaches C3.1
- net GND: now also TP2.1
- net +SOLAR renamed Vin
- new net HIDRV: Q1.1 (G), U1.15 (HIDRV)
- new net SRN: C7.2, R13.2, U1.9 (SRN)
Other:
- note added: "BATT Voltage control"
- note added: "Buck"
- note added: "High-Side Driver Bootstrap"
- note added: "MPPT control"
- note added: "test pads"
- moved on the sheet: C1, C10, C2, C3, C4, C5, C6, C7, C8, C9, D1, D2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
