File: BQ24650_1U_SolarChargerBoard copy.kicad_pcb (KiCad board)
At the start: 2 copper layers, 48 parts, among them J1 Solar IO, J2 Battery IO, J3 CE_MPPSET, Q1 Q_NMOS_GDS, Q2 Q_NMOS_GDS, Q3 Q_NMOS_GDS, U1 BQ24650

Commit message: decided Front and back components
Parts:
- removed TP10, TP11, TP12: TestPoint, TestPoint:TestPoint_Pad_D1.5mm
- added J4: BATT+, Connector_PinHeader_2.54mm:PinHeader_1x01_P2.54mm_Vertical, F.Cu at (122.7, 75.2)
- added J5: BATT-, Connector_PinHeader_2.54mm:PinHeader_1x01_P2.54mm_Vertical, F.Cu at (122.7, 95.7)
- added J6: TS, Connector_PinHeader_2.54mm:PinHeader_1x01_P2.54mm_Vertical, F.Cu at (173.1, 66.8)
- C1, C6, C8, C9: footprint Capacitor_SMD:C_1210_3225Metric -> Capacitor_SMD:C_0805_2012Metric
- J1: value Solar IO -> CE_MPPSET; footprint Connector_PinHeader_2.54mm:PinHeader_1x02_P2.54mm_Vertical -> Connector_PinHeader_2.54mm:PinHeader_1x01_P2.54mm_Vertical
- J2: value Battery IO -> solar+; footprint Connector_PinHeader_2.54mm:PinHeader_1x03_P2.54mm_Vertical -> Connector_PinHeader_2.54mm:PinHeader_1x01_P2.54mm_Vertical
- J3: value CE_MPPSET -> solar-
- R12: footprint Resistor_SMD:R_1206_3216Metric -> Resistor_SMD:R_2512_6332Metric
- moved R5 194.9 mm to (227.9, 99.7)
- moved Q1 184.4 mm to (227.5, 83.7)
- moved Q2 183.9 mm to (227.5, 90.3)
- moved R12 178.1 mm to (227.9, 104.6)
- moved TP1 164.2 mm to (195.7, 60.7)
- moved TP2 164.2 mm to (195.7, 64.2)
- moved TP3 164.2 mm to (195.7, 67.8)
- moved TP7 164.2 mm to (202.8, 60.7)
- moved TP8 164.2 mm to (202.8, 64.2)
- moved TP9 164.2 mm to (202.8, 67.8)
- moved TP4 164.2 mm to (199.3, 60.7)
- moved TP5 164.2 mm to (199.3, 64.2)
- moved TP6 164.2 mm to (199.3, 67.8)
- moved D2 157.3 mm to (204.5, 100.5)
- moved Q3 157.3 mm to (204.5, 105.0)
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Connections:
- J1 pad 1: Vin -> CE
- J2 pad 1: SRN -> Vin
- J3 pad 1: CE -> GND
- TP3 pad 1: CE -> Net-(R4-Pad2)
- TP4 pad 1: STAT1 -> Net-(R1-Pad1)
- TP5 pad 1: STAT2 -> PH
- TP9 pad 1: TERM_EN -> VFB
Other:
- board text added: "Front board"
- board text added: "can be on the Back side, if there is less space"
- board text added: "things to be on the edge or accessible"
