File: BQ24650_1U_SolarChargerBoard copy.kicad_pcb (KiCad board)
At the start: 2 copper layers, 33 x 23 mm, 48 parts, among them J1 CE_MPPSET, J2 solar+, J3 solar-, J4 BATT+, J5 BATT-, J6 TS, Q1 Q_NMOS_GDS, Q2 Q_NMOS_GDS, Q3 Q_NMOS_GDS, U1 BQ24650

Commit message: finishing touches
Routing:
- net VCC: track 15.1 -> 16.2 mm
- net Net-(R1-Pad1): vias 1 -> 0
- net GND: vias 27 -> 28
Other:
- board text added: "BATT-"
- board text added: "BQ24650"
- board text added: "Chip Enable"
- board text added: "GND"
- board text added: "IN+"
- board text added: "IN-"
- board text added: "MPPTSET"
- board text added: "PH"
- board text added: "REGN"
- board text added: "STAT1"
- board text added: "STAT2"
- board text added: "Solar Charger Module"
- board text added: "Thermistor"
- board text added: "VCC"
- board text added: "VFB"
- board text added: "Vref"
